File: passives-reflow-test/passives-reflow-test.kicad_pcb (KiCad board)
At the start: 2 copper layers, 35 x 40 mm, 120 parts

Commit message: Update passives-reflow-test to KiCad 8
Other:
- net class Default removed
